Commit message: add transmission related stuff w/o test

File: package_template/urdf/macro_template.xacro (robot description, xacro)
@@ -1,10 +1,10 @@
 <?xml version="1.0" encoding="utf-8"?>
 <robot xmlns:xacro="http://www.ros.org/wiki/xacro">
-  <xacro:property name="description_package"
-    value="$(find package_template_name)" />
-  <xacro:include filename="${description_package}/urdf/utils.xacro" />
   <xacro:macro name="macro_template_name"
     params="prefix:='' parent xyz:='0 0 0' rpy:='0 0 0' sim:=false">
-    <!-- auto generated urdf below -->
+    <xacro:property name="description_package"
+      value="$(find package_template_name)" />
+    <xacro:include filename="${description_package}/urdf/utils.xacro" />
+    <!-- auto generated below -->
     <!-- base_link to body_lift -->
     <joint name="${prefix}macro_template_name_install_joint" type="fixed">
@@ -13,4 +13,9 @@
       <child link="${prefix}root_link_template_name" />
     </joint>
+    <!-- transmission -->
+    <xacro:include filename="${description_package}/urdf/macro_template_name_transmission.xacro" />
+    <xacro:macro_template_name_transmission prefix="${prefix}" interface_name="velocity" />
+    <!-- <xacro:macro_template_name_transmission prefix="${prefix}" interface_name="position" /> -->
+    <!-- <xacro:macro_template_name_transmission prefix="${prefix}" interface_name="effort" /> -->
   </xacro:macro>
 </robot>

File: package_template/urdf/utils.xacro (robot description, xacro)
@@ -246,3 +246,24 @@
     </link>
   </xacro:macro>
+  <!-- ~~~~~~~~~~~~~~~~~~~~~~~~~~~~~~~~~~~~~~~~~~~~~~~~~~~~~~~~~~~~~~ -->
+  <!-- Macro to configure transmission for a joint                    -->
+  <!--                                                                -->
+  <!-- joint_name:     Name of the joint to configure transmission for -->
+  <!-- interface_name: Type of hardware interface (e.g., effort,      -->
+  <!--                 position, velocity)                            -->
+  <!-- reduction:      Mechanical reduction ratio (default: 1)        -->
+  <!-- ~~~~~~~~~~~~~~~~~~~~~~~~~~~~~~~~~~~~~~~~~~~~~~~~~~~~~~~~~~~~~~ -->
+  <xacro:macro name="config_transmission"
+    params="joint_name interface_name reduction:=1">
+    <transmission name="${joint_name}_${interface_name.lower()}_trans">
+      <type>transmission_interface/SimpleTransmission</type>
+      <joint name="${joint_name}">
+        <hardwareInterface>hardware_interface/${interface_name.capitalize()}JointInterface</hardwareInterface>
+      </joint>
+      <actuator name="${joint_name}_motor">
+        <hardwareInterface>hardware_interface/${interface_name.capitalize()}JointInterface</hardwareInterface>
+        <mechanicalReduction>${reduction}</mechanicalReduction>
+      </actuator>
+    </transmission>
+  </xacro:macro>
 </robot>
